Commit message: feat: replace sample vehicle model with Hyundai Ioniq 5

File: launcher/autoware_launch/vehicle/sample_vehicle_launch/sample_vehicle_description/urdf/vehicle.xacro (robot description, xacro)
@@ -8,5 +8,5 @@
       <origin xyz="${vehicle_info['/**']['ros__parameters']['wheel_base']/2.0} 0 0" rpy="${pi/2.0} 0 ${pi}"/>
       <geometry>
-        <mesh filename="package://sample_vehicle_description/mesh/lexus.dae" scale="1 1 1"/>
+        <mesh filename="package://sample_vehicle_description/mesh/ioniq5.dae" scale="1 1 1"/>
       </geometry>
     </visual>
